Commit message: remove unnecessary quote in joint6-tool0 after 6

File: templates/robot_description/robot_srdf_examples.xacro (robot description, xacro)
@@ -25,5 +25,5 @@
       <joint name="${prefix}joint5"/>
       <joint name="${prefix}joint6"/>
-      <joint name="${prefix}joint6"-tool0"/>
+      <joint name="${prefix}joint6-tool0"/>
     </group>
     <!--DISABLE COLLISIONS: By default it is assumed that any link of the robot could potentially come into collision with any other link in the robot. This tag disables collision checking between a specified pair of links. -->
