Commit message: Add more template stuff. Extend docs. Correct typos and issues.

File: templates/robot_description/robot.urdf.xacro (robot description, xacro)
@@ -2,5 +2,6 @@
 <robot xmlns:xacro="http://wiki.ros.org/xacro" name="$ROBOT_NAME$">
   <!-- Use this if parameters are set from the launch file, otherwise delete -->
-  <xacro:arg name="example_arg" default="test" />
+  <xacro:arg name="use_fake_hardware" default="true" />
+  <xacro:arg name="fake_sensor_commands" default="false" />
   <xacro:include filename="$(find $PKG_NAME$)/urdf/$ROBOT_NAME$/$ROBOT_NAME$_macro.xacro"/>
   <xacro:include filename="$(find $PKG_NAME$)/urdf/$ROBOT_NAME$/$ROBOT_NAME$_macro.ros2_control.xacro"/>
@@ -15,4 +16,5 @@
     name="$ROBOT_NAME$"
     prefix=""
-    example_param="$(arg example_arg)" />
+    use_fake_hardware="$(arg use_fake_hardware)"
+    fake_sensor_commands="$(arg fake_sensor_commands)" />
 </robot>

File: templates/robot_description/robot_macro.ros2_control.xacro (robot description, xacro)
@@ -1,11 +1,16 @@
 <?xml version="1.0"?>
 <robot xmlns:xacro="http://wiki.ros.org/xacro">
-  <xacro:macro name="$ROBOT_NAME$_ros2_control" params="name prefix example_param:=^|test">
+  <xacro:macro name="$ROBOT_NAME$_ros2_control" params="name prefix use_fake_hardware:=^|true fake_sensor_commands:=^|false">
     <ros2_control name="${name}" type="system">
       <hardware>
-        <plugin>fake_components/GenericRobot</plugin>
-        <param name="example_param">${example_param}</param>
+        <xacro:if value="${use_fake_hardware}">
+          <plugin>fake_components/GenericRobot</plugin>
+          <param name="fake_sensor_commands">${fake_sensor_commands}</param>
+        </xacro:if>
+        <xacro:unless value="${use_fake_hardware}">
+          <plugin>robot_hardware_inteface/RobotHardwareInteface</plugin>
+        </xacro:unless>
       </hardware>
-      <joint name="${prefix}joint_1">
+      <joint name="${prefix}joint1">
         <command_interface name="position">     <!-- Add/Remove interfaces as needed -->
           <param name="min">-1</param>
@@ -15,6 +20,7 @@
         <state_interface name="velocity"/>
         <state_interface name="acceleration"/>
+        <param name="initial_position">0.0</param>
       </joint>
-      <joint name="${prefix}joint_2">
+      <joint name="${prefix}joint2">
         <command_interface name="position">     <!-- Add/Remove interfaces as needed -->
           <param name="min">-1</param>
@@ -24,6 +30,7 @@
         <state_interface name="velocity"/>
         <state_interface name="acceleration"/>
+        <param name="initial_position">0.0</param>
       </joint>
-      <joint name="${prefix}joint_3">
+      <joint name="${prefix}joint3">
         <command_interface name="position">     <!-- Add/Remove interfaces as needed -->
           <param name="min">-1</param>
@@ -33,6 +40,7 @@
         <state_interface name="velocity"/>
         <state_interface name="acceleration"/>
+        <param name="initial_position">0.0</param>
       </joint>
-      <joint name="${prefix}joint_4">
+      <joint name="${prefix}joint4">
         <command_interface name="position">     <!-- Add/Remove interfaces as needed -->
           <param name="min">-1</param>
@@ -42,6 +50,7 @@
         <state_interface name="velocity"/>
         <state_interface name="acceleration"/>
+        <param name="initial_position">0.0</param>
       </joint>
-      <joint name="${prefix}joint_5">
+      <joint name="${prefix}joint5">
         <command_interface name="position">     <!-- Add/Remove interfaces as needed -->
           <param name="min">-1</param>
@@ -51,6 +60,7 @@
         <state_interface name="velocity"/>
         <state_interface name="acceleration"/>
+        <param name="initial_position">0.0</param>
       </joint>
-      <joint name="${prefix}joint_6">
+      <joint name="${prefix}joint6">
         <command_interface name="position">     <!-- Add/Remove interfaces as needed -->
           <param name="min">-1</param>
@@ -60,4 +70,5 @@
         <state_interface name="velocity"/>
         <state_interface name="acceleration"/>
+        <param name="initial_position">0.0</param>
       </joint>
       <sensor name="tcp_fts_sensor">            <!-- Remove/change sensors as needed -->

File: templates/robot_description/robot_macro.xacro (robot description, xacro)
@@ -25,5 +25,5 @@
     </link>
     <!-- link 1 -->
-    <link name="${prefix}link_1">
+    <link name="${prefix}link1">
       <!-- Default inertial for Gazebo/Ingnition - copy and edit block from 'common.xacro'
            to get more realistic behaviour-->
@@ -33,5 +33,5 @@
         <geometry>
           <cylinder length="0.3" radius="0.15" />
-<!--           <mesh filename="package://$PKG_NAME$/meshes/$ROBOT_NAME$/visual/link_1.dae" /> -->
+<!--           <mesh filename="package://$PKG_NAME$/meshes/$ROBOT_NAME$/visual/link1.dae" /> -->
         </geometry>
       </visual>
@@ -40,10 +40,10 @@
         <geometry>
           <cylinder length="0.3" radius="0.15" />
-<!--           <mesh filename="package://$PKG_NAME$/meshes/$ROBOT_NAME$/collision/link_1.stl" /> -->
+<!--           <mesh filename="package://$PKG_NAME$/meshes/$ROBOT_NAME$/collision/link1.stl" /> -->
         </geometry>
       </collision>
     </link>
     <!-- link 2 -->
-    <link name="${prefix}link_2">
+    <link name="${prefix}link2">
       <!-- Default inertial for Gazebo/Ingnition - copy and edit block from 'common.xacro'
            to get more realistic behaviour-->
@@ -53,5 +53,5 @@
         <geometry>
           <cylinder length="0.8" radius="0.15" />
-<!--           <mesh filename="package://$PKG_NAME$/meshes/$ROBOT_NAME$/visual/link_2.dae" /> -->
+<!--           <mesh filename="package://$PKG_NAME$/meshes/$ROBOT_NAME$/visual/link2.dae" /> -->
         </geometry>
       </visual>
@@ -60,10 +60,10 @@
         <geometry>
           <cylinder length="0.8" radius="0.15" />
-<!--           <mesh filename="package://$PKG_NAME$/meshes/$ROBOT_NAME$/collision/link_2.stl"  /> -->
+<!--           <mesh filename="package://$PKG_NAME$/meshes/$ROBOT_NAME$/collision/link2.stl"  /> -->
         </geometry>
       </collision>
     </link>
     <!-- link 3 -->
-    <link name="${prefix}link_3">
+    <link name="${prefix}link3">
       <!-- Default inertial for Gazebo/Ingnition - copy and edit block from 'common.xacro'
            to get more realistic behaviour-->
@@ -73,5 +73,5 @@
         <geometry>
           <cylinder length="0.5" radius="0.10" />
-<!--           <mesh filename="package://$PKG_NAME$/meshes/$ROBOT_NAME$/visual/link_3.dae" /> -->
+<!--           <mesh filename="package://$PKG_NAME$/meshes/$ROBOT_NAME$/visual/link3.dae" /> -->
         </geometry>
       </visual>
@@ -80,10 +80,10 @@
         <geometry>
           <cylinder length="0.5" radius="0.10" />
-<!--           <mesh filename="package://$PKG_NAME$/meshes/$ROBOT_NAME$/collision/link_3.stl"  /> -->
+<!--           <mesh filename="package://$PKG_NAME$/meshes/$ROBOT_NAME$/collision/link3.stl"  /> -->
         </geometry>
       </collision>
     </link>
     <!-- link 4 -->
-    <link name="${prefix}link_4">
+    <link name="${prefix}link4">
       <!-- Default inertial for Gazebo/Ingnition - copy and edit block from 'common.xacro'
            to get more realistic behaviour-->
@@ -93,5 +93,5 @@
         <geometry>
           <cylinder length="0.1" radius="0.2" />
-<!--           <mesh filename="package://$PKG_NAME$/meshes/$ROBOT_NAME$/visual/link_4.dae" /> -->
+<!--           <mesh filename="package://$PKG_NAME$/meshes/$ROBOT_NAME$/visual/link4.dae" /> -->
         </geometry>
       </visual>
@@ -100,10 +100,10 @@
         <geometry>
           <cylinder length="0.1" radius="0.2" />
-<!--           <mesh filename="package://$PKG_NAME$/meshes/$ROBOT_NAME$/collision/link_4.stl"  /> -->
+<!--           <mesh filename="package://$PKG_NAME$/meshes/$ROBOT_NAME$/collision/link4.stl"  /> -->
         </geometry>
       </collision>
     </link>
     <!-- link 5 -->
-    <link name="${prefix}link_5">
+    <link name="${prefix}link5">
       <!-- Default inertial for Gazebo/Ingnition - copy and edit block from 'common.xacro'
            to get more realistic behaviour-->
@@ -113,5 +113,5 @@
         <geometry>
           <cylinder length="0.2" radius="0.1" />
-<!--           <mesh filename="package://$PKG_NAME$/meshes/$ROBOT_NAME$/visual/link_5.dae" /> -->
+<!--           <mesh filename="package://$PKG_NAME$/meshes/$ROBOT_NAME$/visual/link5.dae" /> -->
         </geometry>
       </visual>
@@ -120,10 +120,10 @@
         <geometry>
           <cylinder length="0.2" radius="0.1" />
-<!--           <mesh filename="package://$PKG_NAME$/meshes/$ROBOT_NAME$/collision/link_5.stl" /> -->
+<!--           <mesh filename="package://$PKG_NAME$/meshes/$ROBOT_NAME$/collision/link5.stl" /> -->
         </geometry>
       </collision>
     </link>
     <!-- link 6 -->
-    <link name="${prefix}link_6">
+    <link name="${prefix}link6">
       <!-- Default inertial for Gazebo/Ingnition - copy and edit block from 'common.xacro'
            to get more realistic behaviour-->
@@ -133,5 +133,5 @@
         <geometry>
           <cylinder length="0.05" radius="0.1" />
-<!--           <mesh filename="package://$PKG_NAME$/meshes/$ROBOT_NAME$/visual/link_6.dae" /> -->
+<!--           <mesh filename="package://$PKG_NAME$/meshes/$ROBOT_NAME$/visual/link6.dae" /> -->
         </geometry>
       </visual>
@@ -140,5 +140,5 @@
         <geometry>
           <cylinder length="0.05" radius="0.1" />
-<!--           <mesh filename="package://$PKG_NAME$/meshes/$ROBOT_NAME$/collision/link_6.stl" /> -->
+<!--           <mesh filename="package://$PKG_NAME$/meshes/$ROBOT_NAME$/collision/link6.stl" /> -->
         </geometry>
       </collision>
@@ -164,54 +164,54 @@
     </joint>
     <!-- joint 1 -->
-    <joint name="${prefix}joint_1" type="revolute">
+    <joint name="${prefix}joint1" type="revolute">
       <origin xyz="0 0 0.3" rpy="${pi} 0 0" />
       <parent link="${prefix}base_link" />
-      <child link="${prefix}link_1" />
+      <child link="${prefix}link1" />
       <axis xyz="0 0 1" />
       <limit effort="0" lower="${radians(-180)}" upper="${radians(180)}" velocity="${radians(180)}" />
     </joint>
     <!-- joint 2 -->
-    <joint name="${prefix}joint_2" type="revolute">
+    <joint name="${prefix}joint2" type="revolute">
       <origin xyz="0 0 0.3" rpy="${pi/2} 0 0" />
-      <parent link="${prefix}link_1" />
-      <child link="${prefix}link_2" />
+      <parent link="${prefix}link1" />
+      <child link="${prefix}link2" />
       <axis xyz="0 0 1" />
       <limit effort="0" lower="${radians(-180)}" upper="${radians(180)}" velocity="${radians(180)}" />
     </joint>
     <!-- joint 3 -->
-    <joint name="${prefix}joint_3" type="revolute">
+    <joint name="${prefix}joint3" type="revolute">
       <origin xyz="0.8 0 0" rpy="0 0 0" />
-      <parent link="${prefix}link_2" />
-      <child link="${prefix}link_3" />
+      <parent link="${prefix}link2" />
+      <child link="${prefix}link3" />
       <axis xyz="0 0 1" />
       <limit effort="0" lower="${radians(-90)}" upper="${radians(180)}" velocity="${radians(270)}" />
     </joint>
     <!-- joint 4 -->
-    <joint name="${prefix}joint_4" type="revolute">
+    <joint name="${prefix}joint4" type="revolute">
       <origin xyz="0 0.1 0" rpy="0 ${-pi/2} 0" />
-      <parent link="${prefix}link_3" />
-      <child link="${prefix}link_4" />
+      <parent link="${prefix}link3" />
+      <child link="${prefix}link4" />
       <axis xyz="0 0 1" />
       <limit effort="0" lower="${radians(-360)}" upper="${radians(360)}" velocity="${radians(360)}" />
     </joint>
     <!-- joint 5 -->
-    <joint name="${prefix}joint_5" type="revolute">
+    <joint name="${prefix}joint5" type="revolute">
       <origin xyz="0 0 -0.1" rpy="0 ${pi/2} 0" />
-      <parent link="${prefix}link_4" />
-      <child link="${prefix}link_5" />
+      <parent link="${prefix}link4" />
+      <child link="${prefix}link5" />
       <axis xyz="0 0 1" />
       <limit effort="0" lower="${radians(-120)}" upper="${radians(120)}" velocity="${radians(540)}" />
     </joint>
     <!-- joint 6 -->
-    <joint name="${prefix}joint_6" type="revolute">
+    <joint name="${prefix}joint6" type="revolute">
       <origin xyz="0 0 0.1" rpy="0 ${-pi/2} 0" />
-      <parent link="${prefix}link_5" />
-      <child link="${prefix}link_6" />
+      <parent link="${prefix}link5" />
+      <child link="${prefix}link6" />
       <axis xyz="0 0 1" />
       <limit effort="0" lower="${radians(-360)}" upper="${radians(360)}" velocity="${radians(720)}" />
     </joint>
     <!-- tool frame - fixed frame -->
-    <joint name="${prefix}joint_6-tool0" type="fixed">
-      <parent link="${prefix}link_6" />
+    <joint name="${prefix}joint6-tool0" type="fixed">
+      <parent link="${prefix}link6" />
       <child link="${prefix}tool0" />
       <origin xyz="0 0 -0.115" rpy="0 ${-pi} ${-pi/2}" />

Commit message: Added also additional templates for controller testing and precommit udpates

File: templates/robot_description/robot.urdf.xacro (robot description, xacro)
@@ -2,5 +2,5 @@
 <robot xmlns:xacro="http://wiki.ros.org/xacro" name="$ROBOT_NAME$">
   <!-- Use this if parameters are set from the launch file, otherwise delete -->
-  <xacro:arg name="use_fake_hardware" default="true" />
+  <xacro:arg name="use_fake_hardware" default="false" />
   <xacro:arg name="fake_sensor_commands" default="false" />
   <xacro:arg name="prefix" default="" />

File: templates/robot_description/robot_macro.ros2_control.xacro (robot description, xacro)
@@ -1,5 +1,5 @@
 <?xml version="1.0" encoding="UTF-8"?>
 <robot xmlns:xacro="http://wiki.ros.org/xacro">
-  <xacro:macro name="$ROBOT_NAME$_ros2_control" params="name prefix use_fake_hardware:=^|true fake_sensor_commands:=^|false">
+  <xacro:macro name="$ROBOT_NAME$_ros2_control" params="name prefix use_fake_hardware:=^|false fake_sensor_commands:=^|false">
     <ros2_control name="${name}" type="system">
       <hardware>

Commit message: Use 'mock' instead of 'fake' in the nomenclature.

File: templates/robot_description/robot.urdf.xacro (robot description, xacro)
@@ -2,6 +2,6 @@
 <robot xmlns:xacro="http://wiki.ros.org/xacro" name="$ROBOT_NAME$">
   <!-- Use this if parameters are set from the launch file, otherwise delete -->
-  <xacro:arg name="use_fake_hardware" default="false" />
-  <xacro:arg name="fake_sensor_commands" default="false" />
+  <xacro:arg name="use_mock_hardware" default="false" />
+  <xacro:arg name="mock_sensor_commands" default="false" />
   <xacro:arg name="prefix" default="" />
   <xacro:include filename="$(find $PKG_NAME$)/urdf/$ROBOT_NAME$/$ROBOT_NAME$_macro.xacro"/>
@@ -17,5 +17,5 @@
     name="$ROBOT_NAME$"
     prefix="$(arg prefix)"
-    use_fake_hardware="$(arg use_fake_hardware)"
-    fake_sensor_commands="$(arg fake_sensor_commands)" />
+    use_mock_hardware="$(arg use_mock_hardware)"
+    mock_sensor_commands="$(arg mock_sensor_commands)" />
 </robot>

File: templates/robot_description/robot_macro.ros2_control.xacro (robot description, xacro)
@@ -1,13 +1,13 @@
 <?xml version="1.0" encoding="UTF-8"?>
 <robot xmlns:xacro="http://wiki.ros.org/xacro">
-  <xacro:macro name="$ROBOT_NAME$_ros2_control" params="name prefix use_fake_hardware:=^|false fake_sensor_commands:=^|false">
+  <xacro:macro name="$ROBOT_NAME$_ros2_control" params="name prefix use_mock_hardware:=^|false mock_sensor_commands:=^|false">
     <ros2_control name="${name}" type="system">
       <hardware>
-        <xacro:if value="${use_fake_hardware}">
+        <xacro:if value="${use_mock_hardware}">
           <plugin>fake_components/GenericSystem</plugin>
-          <param name="fake_sensor_commands">${fake_sensor_commands}</param>
+          <param name="mock_sensor_commands">${mock_sensor_commands}</param>
           <param name="state_following_offset">0.0</param>
         </xacro:if>
-        <xacro:unless value="${use_fake_hardware}">
+        <xacro:unless value="${use_mock_hardware}">
           <plugin>robot_hardware_inteface/RobotHardwareInteface</plugin>
         </xacro:unless>

Commit message: Updates for the mock HW and Hw Interface things.

File: templates/robot_description/robot.urdf.xacro (robot description, xacro)
@@ -2,7 +2,10 @@
 <robot xmlns:xacro="http://wiki.ros.org/xacro" name="$ROBOT_NAME$">
   <!-- Use this if parameters are set from the launch file, otherwise delete -->
+  <xacro:arg name="prefix" default="" />
   <xacro:arg name="use_mock_hardware" default="false" />
   <xacro:arg name="mock_sensor_commands" default="false" />
-  <xacro:arg name="prefix" default="" />
+  <xacro:arg name="sim_gazebo_classic" default="false" />
+  <xacro:arg name="sim_gazebo" default="false" />
+  <xacro:arg name="simulation_controllers" default="" />
   <xacro:include filename="$(find $PKG_NAME$)/urdf/$ROBOT_NAME$/$ROBOT_NAME$_macro.xacro"/>
   <xacro:include filename="$(find $PKG_NAME$)/urdf/$ROBOT_NAME$/$ROBOT_NAME$_macro.ros2_control.xacro"/>
@@ -18,4 +21,27 @@
     prefix="$(arg prefix)"
     use_mock_hardware="$(arg use_mock_hardware)"
-    mock_sensor_commands="$(arg mock_sensor_commands)" />
+    mock_sensor_commands="$(arg mock_sensor_commands)"
+    sim_gazebo_classic="$(arg sim_gazebo_classic)"
+    sim_gazebo="$(arg sim_gazebo)"/>
+  <xacro:if value="$(arg sim_gazebo_classic)">
+    <!-- Gazebo plugins -->
+    <gazebo reference="world">
+    </gazebo>
+    <gazebo>
+      <plugin filename="libgazebo_ros2_control.so" name="gazebo_ros2_control">
+        <parameters>$(arg simulation_controllers)</parameters>
+      </plugin>
+    </gazebo>
+  </xacro:if>
+  <xacro:if value="$(arg sim_gazebo)">
+    <!-- Gazebo plugins -->
+    <gazebo reference="world">
+    </gazebo>
+    <gazebo>
+      <plugin filename="libign_ros2_control-system.so" name="ign_ros2_control::IgnitionROS2ControlPlugin">
+        <parameters>$(arg simulation_controllers)</parameters>
+        <controller_manager_node_name>$(arg prefix)controller_manager</controller_manager_node_name>
+      </plugin>
+    </gazebo>
+  </xacro:if>
 </robot>

File: templates/robot_description/robot_macro.ros2_control.xacro (robot description, xacro)
@@ -1,13 +1,25 @@
 <?xml version="1.0" encoding="UTF-8"?>
 <robot xmlns:xacro="http://wiki.ros.org/xacro">
-  <xacro:macro name="$ROBOT_NAME$_ros2_control" params="name prefix use_mock_hardware:=^|false mock_sensor_commands:=^|false">
+  <xacro:macro name="$ROBOT_NAME$_ros2_control" params="
+               name
+               prefix
+               use_mock_hardware:=^|false
+               mock_sensor_commands:=^|false
+               sim_gazebo_classic:=^|false
+               sim_gazebo:=^|false"
+               >
     <ros2_control name="${name}" type="system">
       <hardware>
         <xacro:if value="${use_mock_hardware}">
-          <plugin>fake_components/GenericSystem</plugin>
+          <plugin>mock_components/GenericSystem</plugin>
           <param name="mock_sensor_commands">${mock_sensor_commands}</param>
-          <param name="state_following_offset">0.0</param>
         </xacro:if>
-        <xacro:unless value="${use_mock_hardware}">
+        <xacro:if value="${sim_gazebo_classic}">
+          <plugin>gazebo_ros2_control/GazeboSystem</plugin>
+        </xacro:if>
+        <xacro:if value="${sim_gazebo}">
+          <plugin>ign_ros2_control/IgnitionSystem</plugin>
+        </xacro:if>
+        <xacro:unless value="${use_mock_hardware or sim_gazebo_classic or sim_gazebo}">
           <plugin>robot_hardware_inteface/RobotHardwareInteface</plugin>
         </xacro:unless>
@@ -18,8 +30,9 @@
           <param name="max">1</param>
         </command_interface>
-        <state_interface name="position"/>
+        <state_interface name="position">
+          <param name="initial_value">0.0</param>
+        <state_interface/>
         <state_interface name="velocity"/>
         <state_interface name="acceleration"/>
-        <param name="initial_position">0.0</param>
       </joint>
       <joint name="${prefix}joint2">
@@ -28,8 +41,9 @@
           <param name="max">1</param>
         </command_interface>
-        <state_interface name="position"/>
+        <state_interface name="position">
+          <param name="initial_value">0.0</param>
+        <state_interface/>
         <state_interface name="velocity"/>
         <state_interface name="acceleration"/>
-        <param name="initial_position">0.0</param>
       </joint>
       <joint name="${prefix}joint3">
@@ -38,8 +52,9 @@
           <param name="max">1</param>
         </command_interface>
-        <state_interface name="position"/>
+        <state_interface name="position">
+          <param name="initial_value">0.0</param>
+        <state_interface/>
         <state_interface name="velocity"/>
         <state_interface name="acceleration"/>
-        <param name="initial_position">0.0</param>
       </joint>
       <joint name="${prefix}joint4">
@@ -48,8 +63,9 @@
           <param name="max">1</param>
         </command_interface>
-        <state_interface name="position"/>
+        <state_interface name="position">
+          <param name="initial_value">0.0</param>
+        <state_interface/>
         <state_interface name="velocity"/>
         <state_interface name="acceleration"/>
-        <param name="initial_position">0.0</param>
       </joint>
       <joint name="${prefix}joint5">
@@ -58,8 +74,9 @@
           <param name="max">1</param>
         </command_interface>
-        <state_interface name="position"/>
+        <state_interface name="position">
+          <param name="initial_value">0.0</param>
+        <state_interface/>
         <state_interface name="velocity"/>
         <state_interface name="acceleration"/>
-        <param name="initial_position">0.0</param>
       </joint>
       <joint name="${prefix}joint6">
@@ -68,8 +85,9 @@
           <param name="max">1</param>
         </command_interface>
-        <state_interface name="position"/>
+        <state_interface name="position">
+          <param name="initial_value">0.0</param>
+        <state_interface/>
         <state_interface name="velocity"/>
         <state_interface name="acceleration"/>
-        <param name="initial_position">0.0</param>
       </joint>
       <sensor name="tcp_fts_sensor">            <!-- Remove/change sensors as needed -->
