Commit message: Use word 'mock' instead of 'fake' in the nomenclature of ros2_control templates. (#77)
* Use 'mock' instead of 'fake' in the nomenclature.
* Update joint_state_controller name to broadcaster.
* Add launch files for starting simulators.

File: templates/robot_description/robot.urdf.xacro (robot description, xacro)
@@ -2,7 +2,10 @@
 <robot xmlns:xacro="http://wiki.ros.org/xacro" name="$ROBOT_NAME$">
   <!-- Use this if parameters are set from the launch file, otherwise delete -->
-  <xacro:arg name="use_fake_hardware" default="false" />
-  <xacro:arg name="fake_sensor_commands" default="false" />
   <xacro:arg name="prefix" default="" />
+  <xacro:arg name="use_mock_hardware" default="false" />
+  <xacro:arg name="mock_sensor_commands" default="false" />
+  <xacro:arg name="sim_gazebo_classic" default="false" />
+  <xacro:arg name="sim_gazebo" default="false" />
+  <xacro:arg name="simulation_controllers" default="" />
   <xacro:include filename="$(find $PKG_NAME$)/urdf/$ROBOT_NAME$/$ROBOT_NAME$_macro.xacro"/>
   <xacro:include filename="$(find $PKG_NAME$)/urdf/$ROBOT_NAME$/$ROBOT_NAME$_macro.ros2_control.xacro"/>
@@ -17,5 +20,28 @@
     name="$ROBOT_NAME$"
     prefix="$(arg prefix)"
-    use_fake_hardware="$(arg use_fake_hardware)"
-    fake_sensor_commands="$(arg fake_sensor_commands)" />
+    use_mock_hardware="$(arg use_mock_hardware)"
+    mock_sensor_commands="$(arg mock_sensor_commands)"
+    sim_gazebo_classic="$(arg sim_gazebo_classic)"
+    sim_gazebo="$(arg sim_gazebo)"/>
+  <xacro:if value="$(arg sim_gazebo_classic)">
+    <!-- Gazebo plugins -->
+    <gazebo reference="world">
+    </gazebo>
+    <gazebo>
+      <plugin filename="libgazebo_ros2_control.so" name="gazebo_ros2_control">
+        <parameters>$(arg simulation_controllers)</parameters>
+      </plugin>
+    </gazebo>
+  </xacro:if>
+  <xacro:if value="$(arg sim_gazebo)">
+    <!-- Gazebo plugins -->
+    <gazebo reference="world">
+    </gazebo>
+    <gazebo>
+      <plugin filename="libign_ros2_control-system.so" name="ign_ros2_control::IgnitionROS2ControlPlugin">
+        <parameters>$(arg simulation_controllers)</parameters>
+        <controller_manager_node_name>$(arg prefix)controller_manager</controller_manager_node_name>
+      </plugin>
+    </gazebo>
+  </xacro:if>
 </robot>

File: templates/robot_description/robot_macro.ros2_control.xacro (robot description, xacro)
@@ -1,13 +1,25 @@
 <?xml version="1.0" encoding="UTF-8"?>
 <robot xmlns:xacro="http://wiki.ros.org/xacro">
-  <xacro:macro name="$ROBOT_NAME$_ros2_control" params="name prefix use_fake_hardware:=^|false fake_sensor_commands:=^|false">
+  <xacro:macro name="$ROBOT_NAME$_ros2_control" params="
+               name
+               prefix
+               use_mock_hardware:=^|false
+               mock_sensor_commands:=^|false
+               sim_gazebo_classic:=^|false
+               sim_gazebo:=^|false"
+               >
     <ros2_control name="${name}" type="system">
       <hardware>
-        <xacro:if value="${use_fake_hardware}">
-          <plugin>fake_components/GenericSystem</plugin>
-          <param name="fake_sensor_commands">${fake_sensor_commands}</param>
-          <param name="state_following_offset">0.0</param>
+        <xacro:if value="${use_mock_hardware}">
+          <plugin>mock_components/GenericSystem</plugin>
+          <param name="mock_sensor_commands">${mock_sensor_commands}</param>
         </xacro:if>
-        <xacro:unless value="${use_fake_hardware}">
+        <xacro:if value="${sim_gazebo_classic}">
+          <plugin>gazebo_ros2_control/GazeboSystem</plugin>
+        </xacro:if>
+        <xacro:if value="${sim_gazebo}">
+          <plugin>ign_ros2_control/IgnitionSystem</plugin>
+        </xacro:if>
+        <xacro:unless value="${use_mock_hardware or sim_gazebo_classic or sim_gazebo}">
           <plugin>robot_hardware_inteface/RobotHardwareInteface</plugin>
         </xacro:unless>
@@ -18,8 +30,9 @@
           <param name="max">1</param>
         </command_interface>
-        <state_interface name="position"/>
+        <state_interface name="position">
+          <param name="initial_value">0.0</param>
+        <state_interface/>
         <state_interface name="velocity"/>
         <state_interface name="acceleration"/>
-        <param name="initial_position">0.0</param>
       </joint>
       <joint name="${prefix}joint2">
@@ -28,8 +41,9 @@
           <param name="max">1</param>
         </command_interface>
-        <state_interface name="position"/>
+        <state_interface name="position">
+          <param name="initial_value">0.0</param>
+        <state_interface/>
         <state_interface name="velocity"/>
         <state_interface name="acceleration"/>
-        <param name="initial_position">0.0</param>
       </joint>
       <joint name="${prefix}joint3">
@@ -38,8 +52,9 @@
           <param name="max">1</param>
         </command_interface>
-        <state_interface name="position"/>
+        <state_interface name="position">
+          <param name="initial_value">0.0</param>
+        <state_interface/>
         <state_interface name="velocity"/>
         <state_interface name="acceleration"/>
-        <param name="initial_position">0.0</param>
       </joint>
       <joint name="${prefix}joint4">
@@ -48,8 +63,9 @@
           <param name="max">1</param>
         </command_interface>
-        <state_interface name="position"/>
+        <state_interface name="position">
+          <param name="initial_value">0.0</param>
+        <state_interface/>
         <state_interface name="velocity"/>
         <state_interface name="acceleration"/>
-        <param name="initial_position">0.0</param>
       </joint>
       <joint name="${prefix}joint5">
@@ -58,8 +74,9 @@
           <param name="max">1</param>
         </command_interface>
-        <state_interface name="position"/>
+        <state_interface name="position">
+          <param name="initial_value">0.0</param>
+        <state_interface/>
         <state_interface name="velocity"/>
         <state_interface name="acceleration"/>
-        <param name="initial_position">0.0</param>
       </joint>
       <joint name="${prefix}joint6">
@@ -68,8 +85,9 @@
           <param name="max">1</param>
         </command_interface>
-        <state_interface name="position"/>
+        <state_interface name="position">
+          <param name="initial_value">0.0</param>
+        <state_interface/>
         <state_interface name="velocity"/>
         <state_interface name="acceleration"/>
-        <param name="initial_position">0.0</param>
       </joint>
       <sensor name="tcp_fts_sensor">            <!-- Remove/change sensors as needed -->

Commit message: adjust existing description files
* lift robot so it does not clip to ground plane in sim
* new joint position for joint2, same reason as above

File: templates/robot_description/robot.urdf.xacro (robot description, xacro)
@@ -15,5 +15,5 @@
   <!-- set prefix if multiple robots are used -->
   <xacro:$ROBOT_NAME$ prefix="$(arg prefix)" parent="world" >
-    <origin xyz="0 0 0" rpy="0 0 0" />          <!-- position robot in the world -->
+    <origin xyz="0 0 0.1" rpy="0 0 0" />   <!-- to prevent clipping in ground plane in simulation -->
   </xacro:$ROBOT_NAME$>
   <xacro:$ROBOT_NAME$_ros2_control

File: templates/robot_description/robot_macro.xacro (robot description, xacro)
@@ -182,5 +182,5 @@
     <!-- joint 2 -->
     <joint name="${prefix}joint2" type="revolute">
-      <origin xyz="0 0 0.3" rpy="${pi/2} 0 0" />
+      <origin xyz="0 0 0.3" rpy="${pi/2} ${pi/2} 0" />
       <parent link="${prefix}link1" />
       <child link="${prefix}link2" />

Commit message: minor template adjustments

File: templates/robot_description/robot.urdf.xacro (robot description, xacro)
@@ -15,5 +15,5 @@
   <!-- set prefix if multiple robots are used -->
   <xacro:$ROBOT_NAME$ prefix="$(arg prefix)" parent="world" >
-    <origin xyz="0 0 0.1" rpy="0 0 0" />   <!-- to prevent clipping in ground plane in simulation -->
+    <origin xyz="0 0 0.15" rpy="0 0 0" />   <!-- to prevent clipping in ground plane in simulation -->
   </xacro:$ROBOT_NAME$>
   <xacro:$ROBOT_NAME$_ros2_control

Commit message: issue [202]: add pathing flag for gazebo
* during simulation, absolute file:// is used
* on actual robot, relative package:// is used

File: templates/robot_description/robot.urdf.xacro (robot description, xacro)
@@ -14,6 +14,9 @@
   <!-- Load robot's macro with parameters -->
   <!-- set prefix if multiple robots are used -->
-  <xacro:$ROBOT_NAME$ prefix="$(arg prefix)" parent="world" >
-    <origin xyz="0 0 0.15" rpy="0 0 0" />   <!-- to prevent clipping in ground plane in simulation -->
+  <xacro:$ROBOT_NAME$
+    prefix="$(arg prefix)"
+    parent="world"
+    sim_gazebo="$(arg sim_gazebo)">
+    <origin xyz="0 0 0.15" rpy="0 0 0" />          <!-- position robot in the world -->
   </xacro:$ROBOT_NAME$>
   <xacro:$ROBOT_NAME$_ros2_control

File: templates/robot_description/robot_macro.xacro (robot description, xacro)
@@ -3,5 +3,18 @@
   <xacro:include filename="$(find $PKG_NAME$)/urdf/common/inertials.xacro" />
   <xacro:include filename="$(find $PKG_NAME$)/urdf/common/materials.xacro" />
-  <xacro:macro name="$ROBOT_NAME$" params="prefix parent *origin">
+  <xacro:macro name="$ROBOT_NAME$" params="prefix parent sim_gazebo *origin">
+    <!-- determine pathing for gazebo resources -->
+    <xacro:if value="${sim_gazebo}">
+      <xacro:property
+        name="file_prefix"
+        value="file://$(find $PKG_NAME$)"
+        />
+    </xacro:if>
+    <xacro:unless value="${sim_gazebo}">
+      <xacro:property
+        name="file_prefix"
+        value="package://$PKG_NAME$"
+      />
+    </xacro:unless>
     <!-- LINKS -->
     <!-- base link -->
@@ -14,5 +27,5 @@
         <geometry>
           <cylinder length="0.3" radius="0.3" />
-<!--           <mesh filename="package://$PKG_NAME$/meshes/$ROBOT_NAME$/visual/base_link.dae" /> -->
+<!--          <mesh filename="${file_prefix}/meshes/$ROBOT_NAME$/visual/base_link.dae"-->
         </geometry>
         <material name="black"/>
@@ -22,5 +35,5 @@
         <geometry>
           <cylinder length="0.3" radius="0.3" />
-<!--           <mesh filename="package://$PKG_NAME$/meshes/$ROBOT_NAME$/collision/base_link.stl" /> -->
+<!--          <mesh filename="${file_prefix}/meshes/$ROBOT_NAME$/collision/base_link.stl" />-->
         </geometry>
       </collision>
@@ -35,5 +48,5 @@
         <geometry>
           <cylinder length="0.3" radius="0.15" />
-<!--           <mesh filename="package://$PKG_NAME$/meshes/$ROBOT_NAME$/visual/link1.dae" /> -->
+<!--           <mesh filename="${file_prefix}/meshes/$ROBOT_NAME$/visual/link1.dae" /> -->
         </geometry>
         <material name="blue"/>
@@ -43,5 +56,5 @@
         <geometry>
           <cylinder length="0.3" radius="0.15" />
-<!--           <mesh filename="package://$PKG_NAME$/meshes/$ROBOT_NAME$/collision/link1.stl" /> -->
+<!--           <mesh filename="${file_prefix}/meshes/$ROBOT_NAME$/collision/link1.stl" /> -->
         </geometry>
         <material name="green"/>
@@ -57,5 +70,5 @@
         <geometry>
           <cylinder length="0.8" radius="0.15" />
-<!--           <mesh filename="package://$PKG_NAME$/meshes/$ROBOT_NAME$/visual/link2.dae" /> -->
+<!--           <mesh filename="${file_prefix}/meshes/$ROBOT_NAME$/visual/link2.dae" /> -->
         </geometry>
         <material name="grey"/>
@@ -65,5 +78,5 @@
         <geometry>
           <cylinder length="0.8" radius="0.15" />
-<!--           <mesh filename="package://$PKG_NAME$/meshes/$ROBOT_NAME$/collision/link2.stl"  /> -->
+<!--           <mesh filename="${file_prefix}/meshes/$ROBOT_NAME$/collision/link2.stl"  /> -->
         </geometry>
       </collision>
@@ -78,5 +91,5 @@
         <geometry>
           <cylinder length="0.5" radius="0.10" />
-<!--           <mesh filename="package://$PKG_NAME$/meshes/$ROBOT_NAME$/visual/link3.dae" /> -->
+<!--           <mesh filename="${file_prefix}/meshes/$ROBOT_NAME$/visual/link3.dae" /> -->
         </geometry>
         <material name="orange"/>
@@ -86,5 +99,5 @@
         <geometry>
           <cylinder length="0.5" radius="0.10" />
-<!--           <mesh filename="package://$PKG_NAME$/meshes/$ROBOT_NAME$/collision/link3.stl"  /> -->
+<!--           <mesh filename="${file_prefix}/meshes/$ROBOT_NAME$/collision/link3.stl"  /> -->
         </geometry>
       </collision>
@@ -99,5 +112,5 @@
         <geometry>
           <cylinder length="0.1" radius="0.2" />
-<!--           <mesh filename="package://$PKG_NAME$/meshes/$ROBOT_NAME$/visual/link4.dae" /> -->
+<!--           <mesh filename="${file_prefix}/meshes/$ROBOT_NAME$/visual/link4.dae" /> -->
         </geometry>
         <material name="brown"/>
@@ -107,5 +120,5 @@
         <geometry>
           <cylinder length="0.1" radius="0.2" />
-<!--           <mesh filename="package://$PKG_NAME$/meshes/$ROBOT_NAME$/collision/link4.stl"  /> -->
+<!--           <mesh filename="${file_prefix}/meshes/$ROBOT_NAME$/collision/link4.stl"  /> -->
         </geometry>
       </collision>
@@ -120,5 +133,5 @@
         <geometry>
           <cylinder length="0.2" radius="0.1" />
-<!--           <mesh filename="package://$PKG_NAME$/meshes/$ROBOT_NAME$/visual/link5.dae" /> -->
+<!--           <mesh filename="${file_prefix}/meshes/$ROBOT_NAME$/visual/link5.dae" /> -->
         </geometry>
         <material name="red"/>
@@ -128,5 +141,5 @@
         <geometry>
           <cylinder length="0.2" radius="0.1" />
-<!--           <mesh filename="package://$PKG_NAME$/meshes/$ROBOT_NAME$/collision/link5.stl" /> -->
+<!--           <mesh filename="${file_prefix}/meshes/$ROBOT_NAME$/collision/link5.stl" /> -->
         </geometry>
       </collision>
@@ -141,5 +154,5 @@
         <geometry>
           <cylinder length="0.05" radius="0.1" />
-<!--           <mesh filename="package://$PKG_NAME$/meshes/$ROBOT_NAME$/visual/link6.dae" /> -->
+<!--           <mesh filename="${file_prefix}/meshes/$ROBOT_NAME$/visual/link6.dae" /> -->
         </geometry>
         <material name="white"/>
@@ -149,5 +162,5 @@
         <geometry>
           <cylinder length="0.05" radius="0.1" />
-<!--           <mesh filename="package://$PKG_NAME$/meshes/$ROBOT_NAME$/collision/link6.stl" /> -->
+<!--           <mesh filename="${file_prefix}/meshes/$ROBOT_NAME$/collision/link6.stl" /> -->
         </geometry>
       </collision>
