Commit message: add variable names to template files for SED-ing

File: templates/moveit/robot.srdf.xacro (robot description, xacro)
@@ -1,6 +1,6 @@
 <?xml version="1.0" encoding="UTF-8"?>
-<robot xmlns:xacro="http://wiki.ros.org/xacro" name="myrobot">
+<robot xmlns:xacro="http://wiki.ros.org/xacro" name="$ROBOT_NAME$">
   <xacro:arg name="prefix" default="" />
-  <xacro:include filename="$(find myrobot_moveit)/srdf/myrobot_macro.srdf.xacro"/>
-  <xacro:myrobot_srdf prefix="$(arg prefix)"/>
+  <xacro:include filename="$(find $PKG_NAME$)/srdf/$ROBOT_NAME$_macro.srdf.xacro"/>
+  <xacro:$ROBOT_NAME$_srdf prefix="$(arg prefix)"/>
 </robot>

File: templates/moveit/robot_macro.srdf.xacro (robot description, xacro)
@@ -1,7 +1,7 @@
 <?xml version="1.0" encoding="UTF-8"?>
 <robot xmlns:xacro="http://wiki.ros.org/xacro">
-  <xacro:macro name="myrobot_srdf" params="prefix">
+  <xacro:macro name="$ROBOT_NAME$_srdf" params="prefix">
         <!--GROUPS: Representation of a set of joints and links. This can be useful for specifying DOF to plan for, defining arms, end effectors, etc-->
-        <group name="myrobot_manipulator">
+        <group name="${prefix}$ROBOT_NAME$_manipulator">
             <chain base_link="${prefix}base_link" tip_link="${prefix}tool0"/>
         </group>
